File: pcb/Tapper.sch (KiCad schematic (older format))
At the start: 61 parts, among them J1 Barrel_Jack, J2 Conn_01x06_MountingPin, J3 Conn_01x06_MountingPin, J4 Conn_01x06_MountingPin, J5 Conn_01x14, U1 L7805

Commit message: Fix errors in rev1
Parts:
- added R2: 10k, Resistor_SMD:R_1206_3216Metric_Pad1.42x1.75mm_HandSolder, symbol Device:R_Small_US
Connections:
- net +3V3: now also R2.1
- net DISP_RST: now also R2.2
Other:
- moved on the sheet: R1, TP10, TP5
Changed lines of the file:
@@
 encoding utf-8
 Sheet 1 1
-Title ""
-Date ""
-Rev ""
+Title "Tapper Schematic"
+Date "11/01/2020"
+Rev "1"
 Comp ""
 Comment1 ""
@@
 L Connector:TestPoint TP5
 U 1 1 5FC31BB6
-P 5950 4550
-F 0 "TP5" V 6053 4622 50  0000 C CNN
-F 1 "TP" V 5995 4738 50  0001 L CNN
-F 2 "TapperFootprints:SolderPoint" H 6150 4550 50  0001 C CNN
-F 3 "~" H 6150 4550 50  0001 C CNN
-	1    5950 4550
+P 5850 4550
+F 0 "TP5" V 5953 4622 50  0000 C CNN
+F 1 "TP" V 5895 4738 50  0001 L CNN
+F 2 "TapperFootprints:SolderPoint" H 6050 4550 50  0001 C CNN
+F 3 "~" H 6050 4550 50  0001 C CNN
+	1    5850 4550
 	0    -1   -1   0
 $EndComp
@@
 L Device:R_Small_US R1
 U 1 1 5FC32F57
-P 6000 4350
-F 0 "R1" H 6068 4396 50  0000 L CNN
-F 1 "10k" H 6068 4305 50  0000 L CNN
-F 2 "Resistor_SMD:R_1206_3216Metric_Pad1.42x1.75mm_HandSolder" H 6000 4350 50  0001 C CNN
-F 3 "~" H 6000 4350 50  0001 C CNN
-	1    6000 4350
-	1    0    0    -1
-$EndComp
-Wire Wire Line
-	5950 4550 6000 4550
-Wire Wire Line
-	6000 4450 6000 4550
-Connection ~ 6000 4550
-Wire Wire Line
-	6000 4550 6950 4550
+P 5900 4350
+F 0 "R1" H 5968 4396 50  0000 L CNN
+F 1 "10k" H 5968 4305 50  0000 L CNN
+F 2 "Resistor_SMD:R_1206_3216Metric_Pad1.42x1.75mm_HandSolder" H 5900 4350 50  0001 C CNN
+F 3 "~" H 5900 4350 50  0001 C CNN
+	1    5900 4350
+	1    0    0    -1
+$EndComp
+Wire Wire Line
+	5850 4550 5900 4550
+Wire Wire Line
+	5900 4450 5900 4550
+Connection ~ 5900 4550
+Wire Wire Line
+	5900 4550 6950 4550
 $Comp
 L power:+3.3V #PWR01
 U 1 1 5FC442CD
-P 6000 4200
-F 0 "#PWR01" H 6000 4050 50  0001 C CNN
-F 1 "+3.3V" H 6015 4373 50  0000 C CNN
-F 2 "" H 6000 4200 50  0001 C CNN
-F 3 "" H 6000 4200 50  0001 C CNN
-	1    6000 4200
-	1    0    0    -1
-$EndComp
-Wire Wire Line
-	6000 4200 6000 4250
+P 5900 4200
+F 0 "#PWR01" H 5900 4050 50  0001 C CNN
+F 1 "+3.3V" H 5915 4373 50  0000 C CNN
+F 2 "" H 5900 4200 50  0001 C CNN
+F 3 "" H 5900 4200 50  0001 C CNN
+	1    5900 4200
+	1    0    0    -1
+$EndComp
+Wire Wire Line
+	5900 4200 5900 4250
 $Comp
 L Connector:TestPoint TP10
 U 1 1 5FC52053
-P 6400 4150
-F 0 "TP10" V 6503 4222 50  0000 C CNN
-F 1 "TP" V 6445 4338 50  0001 L CNN
-F 2 "TapperFootprints:SolderPoint" H 6600 4150 50  0001 C CNN
-F 3 "~" H 6600 4150 50  0001 C CNN
-	1    6400 4150
-	0    -1   -1   0
-$EndComp
+P 6300 4150
+F 0 "TP10" V 6403 4222 50  0000 C CNN
+F 1 "TP" V 6345 4338 50  0001 L CNN
+F 2 "TapperFootprints:SolderPoint" H 6500 4150 50  0001 C CNN
+F 3 "~" H 6500 4150 50  0001 C CNN
+	1    6300 4150
+	0    -1   -1   0
+$EndComp
+Wire Wire Line
+	6300 4150 6400 4150
+$Comp
+L Device:R_Small_US R2
+U 1 1 5FB7B098
+P 6400 3800
+F 0 "R2" H 6468 3846 50  0000 L CNN
+F 1 "10k" H 6468 3755 50  0000 L CNN
+F 2 "Resistor_SMD:R_1206_3216Metric_Pad1.42x1.75mm_HandSolder" H 6400 3800 50  0001 C CNN
+F 3 "~" H 6400 3800 50  0001 C CNN
+	1    6400 3800
+	1    0    0    -1
+$EndComp
+Wire Wire Line
+	6400 3900 6400 4150
+Connection ~ 6400 4150
 Wire Wire Line
 	6400 4150 6950 4150
+$Comp
+L power:+3.3V #PWR?
+U 1 1 5FBB2430
+P 6400 3650
+F 0 "#PWR?" H 6400 3500 50  0001 C CNN
+F 1 "+3.3V" H 6415 3823 50  0000 C CNN
+F 2 "" H 6400 3650 50  0001 C CNN
+F 3 "" H 6400 3650 50  0001 C CNN
+	1    6400 3650
+	1    0    0    -1
+$EndComp
+Wire Wire Line
+	6400 3650 6400 3700
 $EndSCHEMATC
